File: nand-flash-eval.kicad_pcb (KiCad board)
At the start: 2 copper layers, 16 parts, among them J1 FH26-45S-0.3SHW, J2 PinSocket_2.54mm, J3 Conn_UART, J4 Conn_MISC, U1 TC58BVG0S3HTA00, U2 TC58BVG0S3HTA00

Commit message: feat(wip): IO0-7配線
Parts:
- C2, C4: value 10u -> 0.1u
- moved C3 35.5 mm to (93.6, 94.3), turned to -90 degrees
- moved C1 31.0 mm to (94.0, 68.9), turned to -90 degrees
- moved C4 19.4 mm to (120.0, 94.3), turned to -90 degrees
- moved C2 10.6 mm to (119.4, 68.9), turned to -90 degrees
Routing:
- net GND: track 104.3 -> 307.7 mm, vias 13 -> 8
- net /IO1: track 0.00 -> 123.2 mm, vias 0 -> 5
- net /MISC1: track 136.9 -> 33.3 mm, vias 0 -> 1
- net /UART_TX: track 126.4 -> 28.0 mm, vias 0 -> 1
- net /IO3: track 22.6 -> 113.9 mm, vias 0 -> 4
- net /RY/BY#: track 119.0 -> 28.7 mm, vias 0 -> 1
- net /IO2: track 24.3 -> 113.3 mm, vias 0 -> 4
- net /IO7: track 17.1 -> 105.9 mm, vias 0 -> 4
- net /IO6: track 19.0 -> 107.1 mm, vias 0 -> 4
- net /WP#: track 107.1 -> 26.6 mm, vias 0 -> 1
- net /ALE: track 99.6 -> 27.6 mm, vias 0 -> 1
- net /CE0#: track 90.1 -> 29.2 mm, vias 0 -> 1
- net /IO4: track 60.7 -> 120.5 mm, vias 0 -> 5
- net /IO5: track 67.8 -> 120.0 mm, vias 0 -> 5
- net /MISC6: track 0.00 -> 39.0 mm, vias 0 -> 1
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