File: nand-flash-eval.kicad_sch (KiCad schematic)
At the start: 0 parts

Commit message: feat: create TC58BVG0S3HTA00 symbol
Parts:
- added U1: TC58BVG0S3HTA00, Package_SO:TSOP-I-48_18.4x12mm_P0.5mm, symbol nand-flash-eval:TC58BVG0S3HTA00
Changed lines of the file:
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@@
 	(generator_version "9.0")
 	(paper "A4")
+	(symbol
+		(lib_id "nand-flash-eval:TC58BVG0S3HTA00")
+		(at 129.54 104.14 0)
+		(unit 1)
+		(exclude_from_sim no)
+		(in_bom yes)
+		(on_board yes)
+		(dnp no)
+		(fields_autoplaced yes)
+		(property "Reference" "U1"
+			(at 138.43 49.53 0)
+			(effects
+				(font
+					(size 1.27 1.27)
+				)
+			)
+		)
+		(property "Value" "TC58BVG0S3HTA00"
+			(at 138.43 52.07 0)
+			(effects
+				(font
+					(size 1.27 1.27)
+				)
+			)
+		)
+		(property "Footprint" "Package_SO:TSOP-I-48_18.4x12mm_P0.5mm"
+			(at 129.286 110.744 0)
+			(effects
+				(font
+					(size 1.27 1.27)
+				)
+				(hide yes)
+			)
+		)
+		(property "Datasheet" "https://www.kioxia.com/ja-jp/business/memory/slc-nand/detail.TC58BVG0S3HTA00.html"
+			(at 135.89 108.458 0)
+			(effects
+				(font
+					(size 1.27 1.27)
+				)
+				(hide yes)
+			)
+		)
+		(property "Description" "https://www.kioxia.com/ja-jp/business/memory/slc-nand/detail.TC58BVG0S3HTA00.html"
+			(at 129.54 105.918 0)
+			(effects
+				(font
+					(size 1.27 1.27)
+				)
+				(hide yes)
+			)
+		)
+		(pin "17"
+		)
+		(pin "7"
+		)
+		(pin "19"
+		)
+		(pin "36"
+		)
+		(pin "18"
+		)
+		(pin "29"
+		)
+		(pin "43"
+		)
+		(pin "44"
+		)
+		(pin "30"
+		)
+		(pin "41"
+		)
+		(pin "42"
+		)
+		(pin "31"
+		)
+		(pin "9"
+		)
+		(pin "16"
+		)
+		(pin "32"
+		)
+		(pin "8"
+		)
+		(pin "12"
+		)
+		(pin "37"
+		)
+		(pin "13"
+		)
+		(instances
+			(project ""
+				(path "/8b7b9457-2a92-4e87-8d6b-6a422e047b1a"
+					(reference "U1")
+					(unit 1)
+				)
+			)
+		)
+	)
 	(sheet_instances
 		(path "/"

Commit message: feat: 大体書いた
Parts:
- added C1, C3: 0.1u, Capacitor_SMD:C_0402_1005Metric, symbol Device:C_Small
- added C2, C4: 10u, Capacitor_SMD:C_0402_1005Metric, symbol Device:C_Small
- added J1: FH26-45S-0.3SHW, Connector_FFC-FPC:Hirose_FH26-45S-0.3SHW_2Rows-45Pins-1MP_P0.60mm_Horizontal, symbol Connector_Generic:Conn_02x26_Odd_Even
- added J2: PinSocket_2.54mm, Connector_PinSocket_2.54mm:PinSocket_2x25_P2.54mm_Vertical, symbol Connector_Generic:Conn_02x26_Odd_Even
- added R1, R2: 5k1, symbol Device:R_Small
- added U2: TC58BVG0S3HTA00, Package_SO:TSOP-I-48_18.4x12mm_P0.5mm, symbol nand-flash-eval:TC58BVG0S3HTA00
Connections:
- net +3V3: now reaches U1.12 (VCC)
- net +3V3: now also C1.1, C2.1, C3.1, C4.1, J1.1 (Pin_1), J1.2 (Pin_2), J1.3 (Pin_3), J2.1 (Pin_1), J2.2 (Pin_2), J2.3 (Pin_3), R2.1, U2.12 (VCC)
- net GND: now reaches U1.13 (VSS)
- net GND: now also U1.36 (VSS), C1.2, C2.2, C3.2, C4.2, J1.10 (Pin_10), J1.13 (Pin_13), J1.16 (Pin_16), J1.19 (Pin_19), J1.22 (Pin_22), J1.25 (Pin_25), J1.28 (Pin_28), J1.31 (Pin_31), J1.34 (Pin_34), J1.37 (Pin_37), J1.4 (Pin_4), J1.40 (Pin_40), J1.43 (Pin_43), J1.44 (Pin_44), J1.45 (Pin_45), J1.7 (Pin_7), J2.10 (Pin_10), J2.13 (Pin_13), J2.16 (Pin_16), J2.19 (Pin_19), J2.22 (Pin_22), J2.25 (Pin_25), J2.28 (Pin_28), J2.31 (Pin_31), J2.34 (Pin_34), J2.37 (Pin_37), J2.4 (Pin_4), J2.40 (Pin_40), J2.43 (Pin_43), J2.44 (Pin_44), J2.45 (Pin_45), J2.7 (Pin_7), R1.2, U2.13 (VSS), U2.36 (VSS)
- net CLE: now reaches U1.16 (CLE)
- net CLE: now also J1.20 (Pin_20), J2.20 (Pin_20), U2.16 (CLE)
- net ALE: now reaches U1.17 (ALE)
- net ALE: now also J1.21 (Pin_21), J2.21 (Pin_21), U2.17 (ALE)
- net WE#: now reaches U1.18 (WE#)
- net WE#: now also J1.24 (Pin_24), J2.24 (Pin_24), U2.18 (WE#)
- net WP#: now reaches U1.19 (WP#)
- net WP#: now also J1.23 (Pin_23), J2.23 (Pin_23), R1.1, U2.19 (WP#)
- net IO1: now reaches U1.29 (IO1)
- net IO1: now also J1.5 (Pin_5), J2.5 (Pin_5), U2.29 (IO1)
- net IO2: now reaches U1.30 (IO2)
- net IO2: now also J1.6 (Pin_6), J2.6 (Pin_6), U2.30 (IO2)
- net IO3: now reaches U1.31 (IO3)
- net IO3: now also J1.8 (Pin_8), J2.8 (Pin_8), U2.31 (IO3)
- net IO4: now reaches U1.32 (IO4)
- net IO4: now also J1.9 (Pin_9), J2.9 (Pin_9), U2.32 (IO4)
- net IO5: now reaches U1.41 (IO5)
- net IO5: now also J1.11 (Pin_11), J2.11 (Pin_11), U2.41 (IO5)
- net IO6: now reaches U1.42 (IO6)
- net IO6: now also J1.12 (Pin_12), J2.12 (Pin_12), U2.42 (IO6)
- net IO7: now reaches U1.43 (IO7)
- net IO7: now also J1.14 (Pin_14), J2.14 (Pin_14), U2.43 (IO7)
- net IO8: now reaches U1.44 (IO8)
- net IO8: now also J1.15 (Pin_15), J2.15 (Pin_15), U2.44 (IO8)
- net RY/BY#: now reaches U1.7 (RY/BY#)
- net RY/BY#: now also J1.27 (Pin_27), J2.27 (Pin_27), R2.2, U2.7 (RY/BY#)
- net RE#: now reaches U1.8 (RE#)
- net RE#: now also J1.26 (Pin_26), J2.26 (Pin_26), U2.8 (RE#)
- net CE0#: now reaches U1.9 (CE#)
- net CE0#: now also J1.17 (Pin_17), J2.17 (Pin_17), U2.9 (CE#)
- new net CE1#: J1.18 (Pin_18), J2.18 (Pin_18)
- new net MISC0: J1.32 (Pin_32), J2.32 (Pin_32)
- new net MISC1: J1.33 (Pin_33), J2.33 (Pin_33)
- new net MISC2: J1.35 (Pin_35), J2.35 (Pin_35)
- new net MISC3: J1.36 (Pin_36), J2.36 (Pin_36)
- new net MISC4: J1.38 (Pin_38), J2.38 (Pin_38)
- new net MISC5: J1.39 (Pin_39), J2.39 (Pin_39)
- new net MISC6: J1.41 (Pin_41), J2.41 (Pin_41)
- new net MISC7: J1.42 (Pin_42), J2.42 (Pin_42)
- new net UART_RX: J1.30 (Pin_30), J2.30 (Pin_30)
- new net UART_TX: J1.29 (Pin_29), J2.29 (Pin_29)
- no-connect marks 0 -> 14
Other:
- moved on the sheet: U1

Commit message: feat: ERC Pass
Parts:
- added J3: Conn_UART, Connector_PinSocket_2.54mm:PinSocket_2x04_P2.54mm_Vertical, symbol Connector_Generic:Conn_02x04_Odd_Even
- added J4: Conn_MISC, Connector_PinSocket_2.54mm:PinSocket_2x10_P2.54mm_Vertical, symbol Connector_Generic:Conn_02x10_Odd_Even
Connections:
- net +3V3: now also U1.37 (VCC), U2.37 (VCC), J3.5 (Pin_5), J4.17 (Pin_17)
- net GND: now also J3.2 (Pin_2), J3.4 (Pin_4), J3.6 (Pin_6), J3.7 (Pin_7), J3.8 (Pin_8), J4.10 (Pin_10), J4.12 (Pin_12), J4.14 (Pin_14), J4.16 (Pin_16), J4.18 (Pin_18), J4.19 (Pin_19), J4.2 (Pin_2), J4.20 (Pin_20), J4.4 (Pin_4), J4.6 (Pin_6), J4.8 (Pin_8)
- net MISC0: now also J4.1 (Pin_1)
- net MISC1: now also J4.3 (Pin_3)
- net MISC2: now also J4.5 (Pin_5)
- net MISC3: now also J4.7 (Pin_7)
- net MISC4: now also J4.9 (Pin_9)
- net MISC5: now also J4.11 (Pin_11)
- net MISC6: now also J4.13 (Pin_13)
- net MISC7: now also J4.15 (Pin_15)
- net UART_RX: now also J3.3 (Pin_3)
- net UART_TX: now also J3.1 (Pin_1)
Other:
- company: (none) -> wipeseals
- title: (none) -> nand-flash-eval
- moved on the sheet: J1, J2

Commit message: fix: CE0/1
Connections:
- net CE0#: no longer U2.9 (CE#)
- net CE1#: now also U2.9 (CE#)
Changed lines of the file:
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@@
 		)
 	)
-	(label "CE0#"
+	(label "CE1#"
 		(at 30.48 154.94 0)
 		(effects

Commit message: feat(wip): 配線検討開始
Parts:
- added H1, H2, H3, H4: MountingHole, MountingHole:MountingHole_3.2mm_M3_ISO7380, symbol Mechanical:MountingHole
- R1, R2: footprint (none) -> Resistor_SMD:R_0402_1005Metric

Commit message: feat(wip): IO0-7配線
Parts:
- C2, C4: value 10u -> 0.1u
Changed lines of the file:
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@@
 			)
 		)
-		(property "Value" "10u"
+		(property "Value" "0.1u"
 			(at 93.98 52.0762 0)
 			(effects
@@
 			)
 		)
-		(property "Value" "10u"
+		(property "Value" "0.1u"
 			(at 93.98 138.4362 0)
 			(effects
